Commit message: git push -u origin main --force

File: ur5_robotiq_85.urdf (robot description, URDF)
Before this commit: robot ur5_robotiq_85, 20 links, 19 joints
Links:
- link base_link: geometry collision mesh filename=meshes/ur5/collision/base.stl; visual mesh filename=meshes/ur5/visual/base.obj
- link forearm_link: geometry collision mesh filename=meshes/ur5/collision/forearm.stl; visual mesh filename=meshes/ur5/visual/forearm.obj
- link left_inner_finger: geometry collision mesh filename=meshes/robotiq_85/collision/robotiq_arg2f_85_inner_finger.d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 scale=0.001 0.001 0.001; visual mesh filename=meshes/robotiq_85/visual/robotiq_arg2f_85_inner_finger.dae scale=0.001 0.001 0.001
- link left_inner_knuckle: geometry collision mesh filename=meshes/robotiq_85/collision/robotiq_arg2f_85_inner_knuckle.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 scale=0.001 0.001 0.001; visual mesh filename=meshes/robotiq_85/visual/robotiq_arg2f_85_inner_knuckle.dae scale=0.001 0.001 0.001
- link left_outer_finger: geometry collision mesh filename=meshes/robotiq_85/collision/robotiq_arg2f_85_outer_finger.d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 scale=0.001 0.001 0.001; visual mesh filename=meshes/robotiq_85/visual/robotiq_arg2f_85_outer_finger.dae scale=0.001 0.001 0.001
- link left_outer_knuckle: geometry collision mesh filename=meshes/robotiq_85/collision/robotiq_arg2f_85_outer_knuckle.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 scale=0.001 0.001 0.001; visual mesh filename=meshes/robotiq_85/visual/robotiq_arg2f_85_outer_knuckle.dae scale=0.001 0.001 0.001
- link right_inner_finger: geometry collision mesh filename=meshes/robotiq_85/collision/robotiq_arg2f_85_inner_finger.d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 scale=0.001 0.001 0.001; visual mesh filename=meshes/robotiq_85/visual/robotiq_arg2f_85_inner_finger.dae scale=0.001 0.001 0.001
- link right_inner_knuckle: geometry collision mesh filename=meshes/robotiq_85/collision/robotiq_arg2f_85_inner_knuckle.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 scale=0.001 0.001 0.001; visual mesh filename=meshes/robotiq_85/visual/robotiq_arg2f_85_inner_knuckle.dae scale=0.001 0.001 0.001
- link right_outer_finger: geometry collision mesh filename=meshes/robotiq_85/collision/robotiq_arg2f_85_outer_finger.d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 scale=0.001 0.001 0.001; visual mesh filename=meshes/robotiq_85/visual/robotiq_arg2f_85_outer_finger.dae scale=0.001 0.001 0.001
- link right_outer_knuckle: geometry collision mesh filename=meshes/robotiq_85/collision/robotiq_arg2f_85_outer_knuckle.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 scale=0.001 0.001 0.001; visual mesh filename=meshes/robotiq_85/visual/robotiq_arg2f_85_outer_knuckle.dae scale=0.001 0.001 0.001
- link robotiq_arg2f_base_link: geometry collision mesh filename=meshes/robotiq_85/collision/robotiq_arg2f_base_link.stl; visual mesh filename=meshes/robotiq_85/visual/robotiq_arg2f_85_base_link.dae scale=0.001 0.001 0.001
- link shoulder_link: geometry collision mesh filename=meshes/ur5/collision/shoulder.stl; visual mesh filename=meshes/ur5/visual/shoulder.obj
- link upper_arm_link: geometry collision mesh filename=meshes/ur5/collision/upperarm.stl; visual mesh filename=meshes/ur5/visual/upperarm.obj
- link wrist_1_link: geometry collision mesh filename=meshes/ur5/collision/wrist1.stl; visual mesh filename=meshes/ur5/visual/wrist1.obj
- link wrist_2_link: geometry collision mesh filename=meshes/ur5/collision/wrist2.stl; visual mesh filename=meshes/ur5/visual/wrist2.obj
- link wrist_3_link: geometry collision mesh filename=meshes/ur5/collision/wrist3.stl; visual mesh filename=meshes/ur5/visual/wrist3.obj
